Commit message: # GOAL 4: Add LiDAR Sensor to model

File: src/robot_description/urdf/robot_description.xacro (robot description, xacro)
@@ -7,7 +7,7 @@
 	<link name="base_footprint" />
 	<joint name="base_footprint_joint" type="fixed">
-		<origin xyz="0 0 0.05" rpy="0 0 0" />
-		<parent link="base_footprint" />
-		<child link="base_link" />
+		<origin xyz="0 0 -0.05" rpy="0 0 0" />
+		<parent link="base_link" />
+		<child link="base_footprint" />
 	</joint>
 	<link name="base_link">
@@ -166,4 +166,34 @@
 		</plugin>
 	</gazebo>
+	<gazebo reference="lidar_1">
+		<sensor name="gpu_lidar" type="gpu_lidar">
+			<pose>0 0 0 0 0 0</pose>
+			<topic>lidar</topic>
+			<update_rate>30</update_rate>
+			<frame_id>lidar_1</frame_id>
+			<always_on>true</always_on>
+			<visualize>true</visualize>
+			<ray>
+				<scan>
+					<horizontal>
+						<samples>360</samples>
+						<min_angle>-3.14159</min_angle>
+						<max_angle>3.14159</max_angle>
+					</horizontal>
+				</scan>
+				<range>
+					<min>0.08</min>
+					<max>10.0</max>
+				</range>
+			</ray>
+		</sensor>
+	</gazebo>
+	<gazebo>
+		<plugin
+			filename="gz-sim-sensors-system"
+			name="gz::sim::systems::Sensors">
+			<render_engine>ogre2</render_engine>
+		</plugin>
+	</gazebo>
 	<gazebo reference="left_wheel_1">
 		<mu1>1.0</mu1>

Commit message: removed base_footprint from repo

File: src/robot_description/urdf/robot_description.xacro (robot description, xacro)
@@ -2,13 +2,5 @@
 <robot name="robot_description" xmlns:xacro="http://www.ros.org/wiki/xacro">
 	<xacro:include filename="$(find robot_description)/urdf/materials.xacro" />
-	<xacro:include filename="$(find robot_description)/urdf/robot_description.ros2control" />
 	<xacro:include filename="$(find robot_description)/urdf/robot_description.gazebo" />
-	<!-- Base footprint (planar frame) -->
-	<link name="base_footprint" />
-	<joint name="base_footprint_joint" type="fixed">
-		<origin xyz="0 0 -0.05" rpy="0 0 0" />
-		<parent link="base_link" />
-		<child link="base_footprint" />
-	</joint>
 	<link name="base_link">
 		<inertial>
@@ -167,8 +159,8 @@
 	</gazebo>
 	<gazebo reference="lidar_1">
-		<sensor name="gpu_lidar" type="gpu_lidar">
+		<sensor name="laser" type="gpu_lidar">
 			<pose>0 0 0 0 0 0</pose>
 			<topic>lidar</topic>
-			<update_rate>30</update_rate>
+			<update_rate>20</update_rate>
 			<frame_id>lidar_1</frame_id>
 			<always_on>true</always_on>
@@ -177,5 +169,5 @@
 				<scan>
 					<horizontal>
-						<samples>360</samples>
+						<samples>180</samples>
 						<min_angle>-3.14159</min_angle>
 						<max_angle>3.14159</max_angle>
